File: CIAA-UNO/CIAA-UNO.sch (KiCad schematic (older format))
At the start: 0 parts

Commit message: Modificaciones menores
Se agregó el conector de alimentación, fiduciales y logos. Falta comentarios con datos de fabricación.
Changed lines of the file:
@@
 F3 "ARD_AN5/SCL" I L 7550 5150 60
 F4 "ARD_AN4/SDA" I L 7550 5300 60
-F5 "AREF" I L 7550 2700 60
 F6 "ARD_DIG13/SPI_SCK" I L 7550 2850 60
 F7 "ARD_DIG12/SPI_MISO" I L 7550 3000 60
@@
 $EndSheet
 Wire Wire Line
-	7050 2700 7550 2700
-Wire Wire Line
 	7550 2850 7300 2850
