File: CIAA-UNO/EFM32HG-48LQFP.sch (KiCad schematic (older format))
At the start: 16 parts, among them J2 SWD, SW1 reset, SW2 reset, U5 EFM32HG-48LQFP

Commit message: Diseño del PCB
Faltan fiduciales, comentarios y rótulo.
Changed lines of the file:
@@
 	1875 2400 1800 2400
 Text Label 8250 4700 0    40   ~ 0
-PA10
+PC4
 Text Label 8250 5300 0    40   ~ 0
 PB8

Commit message: Modificaciones menores
Se agregó el conector de alimentación, fiduciales y logos. Falta comentarios con datos de fabricación.
Parts:
- added F1, F2, F3: Fiducial, Fiducial:Fiducial_0.5mm_Dia_1mm_Outer, symbol Mechanical:MountingHole
Connections:
- no-connect marks 0 -> 11
Changed lines of the file:
@@
 Wire Wire Line
 	8325 750  9350 750
+NoConn ~ 3650 2650
+NoConn ~ 3750 2650
+NoConn ~ 4050 2650
+NoConn ~ 4150 2650
+NoConn ~ 4250 2650
+NoConn ~ 2650 3450
+NoConn ~ 2650 3550
+NoConn ~ 2650 3650
+NoConn ~ 3850 5350
+NoConn ~ 4250 5350
+NoConn ~ 5350 3850
+$Comp
+L Mechanical:MountingHole F1
+U 1 1 5BBE0C63
+P 1790 5155
+F 0 "F1" H 1890 5201 50  0000 L CNN
+F 1 "Fiducial" H 1890 5110 50  0000 L CNN
+F 2 "Fiducial:Fiducial_0.5mm_Dia_1mm_Outer" H 1790 5155 50  0001 C CNN
+F 3 "~" H 1790 5155 50  0001 C CNN
+	1    1790 5155
+	1    0    0    -1
+$EndComp
+$Comp
+L Mechanical:MountingHole F2
+U 1 1 5BBE0D63
+P 1790 5535
+F 0 "F2" H 1890 5581 50  0000 L CNN
+F 1 "Fiducial" H 1890 5490 50  0000 L CNN
+F 2 "Fiducial:Fiducial_0.5mm_Dia_1mm_Outer" H 1790 5535 50  0001 C CNN
+F 3 "~" H 1790 5535 50  0001 C CNN
+	1    1790 5535
+	1    0    0    -1
+$EndComp
+$Comp
+L Mechanical:MountingHole F3
+U 1 1 5BBE0E5E
+P 1790 5895
+F 0 "F3" H 1890 5941 50  0000 L CNN
+F 1 "Fiducial" H 1890 5850 50  0000 L CNN
+F 2 "Fiducial:Fiducial_0.5mm_Dia_1mm_Outer" H 1790 5895 50  0001 C CNN
+F 3 "~" H 1790 5895 50  0001 C CNN
+	1    1790 5895
+	1    0    0    -1
+$EndComp
 $EndSCHEMATC

Commit message: Revisión 2
Se tomaron en  cosideración las correcciones y se modificó para cumplir con las consignas.
Parts:
- SW2: value reset -> user
Connections:
- net labels added: 3v3_LDO, USB_VCC
- wire segments 89 -> 60
- no-connect marks 11 -> 14
Other:
- note added: "ANALOG INPUT"
- note added: "DIGITAL PINS / PWM"
- note added: "USB"
